File: Laser_Driver/bigpulse.kicad_sch (KiCad schematic)
At the start: 58 parts, among them IC1 UCC27424P, J1 TRIG, J2 12VIN, J3 BANANA_V+, J4 BANANA_V-, Q1 ZTX415, Q2 ZTX415, Q3 ZTX415, Q4 ZTX415, Q5 STP45N65M5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

Commit message: Minor improvements after prototyping
Legs of MOSFET were switched.
Connections:
- net TRIG1: now also Q5.1 (G); no longer Q5.2 (G)
- net at C2.1, C3.1, C4.1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: now also Q5.2 (D); no longer Q5.1 (D)
