File: R00 Driver/00 - Laser_Driver/bigpulse.kicad_sch (KiCad schematic)
At the start: 58 parts, among them IC1 UCC27424P, J1 TRIG, J2 12VIN, J3 BANANA_V+, J4 BANANA_V-, Q1 ZTX415, Q2 ZTX415, Q3 ZTX415, Q4 ZTX415, Q5 STP45N65M5, U1 LT8365

Commit message: Added the design of the new single-laser double-pulse driver (R01)
This is a major revision. The R01 driver is now our new workhorse in our lab. It not only saves an entire laser, but has greatly improved thermal performance.
Parts:
- C1, C14, C15, C16, C17, C18, C19, C2, C20, C21, C3, C4, C5, C6, C7, C8, L1: LCSC (none) -> C95843
- D1: LCSC (none) -> C70426
- D2, D3, D4, D5, D6: LCSC (none) -> C156325
- IC1: LCSC (none) -> C72129
- J1, TP1: LCSC (none) -> C3172499
- Q5: LCSC (none) -> C672233
- R1, R12, R2, R20, R26, R27, R28, R3, R4, R5, R6, R7, R8, RV1, RV2: LCSC (none) -> C719184
- R14, R19, R23, R24, R25: LCSC (none) -> C335092
- U1: LCSC (none) -> C673785
