File: R01 Driver/01 - Laser_Driver R01/DoublePulse.kicad_pcb (KiCad board)
At the start: 4 copper layers, 84.1 x 60.6 mm, 73 parts, among them IC1 UCC27424P, J1 TRIG, J2 12VIN, J3 TRIG, Q1 STP45N65M5, Q2 STP45N65M5, U1 LT8365

Commit message: Small updates
Other:
- board text added: "18V 0.1A"
Changed lines of the file:
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@@
 		(layer "Edge.Cuts")
+	)
+	(gr_text "18V\n0.1A"
+		(at 146.84 102.28 0)
+		(layer "F.SilkS")
+		(effects
+			(font
+				(size 1 0.9)
+				(thickness 0.18)
+				(bold yes)
+			)
+			(justify right)
+		)
 	)
 	(gr_text "Schlieren Dual\nPulsed Driver\nRev. Sep 26"
